File: production/ecad/KiCad/Lodcell_Bryan/Lodcell_Bryan.kicad_sch (KiCad schematic)
At the start: 24 parts, among them J1 LoadCellConnector, J2 power_for_Loadcell, J3 ConnToESP32, U1 ADS1231IDR, U2 TXB0104DR

Commit message: Improved differential signals. switched to 2 layer board
Parts:
- renumbered R2 to R1, R3 to R2, R4 to R3, R1 to R4
Changed lines of the file:
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@@
 		(on_board yes)
 		(dnp no)
-		(property "Reference" "R4"
+		(property "Reference" "R3"
 			(at 52.07 189.738 90)
 			(effects
@@
 			(project "Lodcell_Bryan"
 				(path "/3f57d594-36f2-42e1-9017-f4e9011de5a2"
-					(reference "R4")
+					(reference "R3")
 					(unit 1)
 				)
@@
 		(on_board yes)
 		(dnp no)
-		(property "Reference" "R1"
+		(property "Reference" "R4"
 			(at 41.91 165.608 90)
 			(effects
@@
 			(project "Lodcell_Bryan"
 				(path "/3f57d594-36f2-42e1-9017-f4e9011de5a2"
-					(reference "R1")
+					(reference "R4")
 					(unit 1)
 				)
@@
 		(on_board yes)
 		(dnp no)
-		(property "Reference" "R2"
+		(property "Reference" "R1"
 			(at 35.56 149.098 90)
 			(effects
@@
 			(project "Lodcell_Bryan"
 				(path "/3f57d594-36f2-42e1-9017-f4e9011de5a2"
-					(reference "R2")
+					(reference "R1")
 					(unit 1)
 				)
@@
 		(on_board yes)
 		(dnp no)
-		(property "Reference" "R3"
+		(property "Reference" "R2"
 			(at 46.99 173.99 90)
 			(effects
@@
 			(project "Lodcell_Bryan"
 				(path "/3f57d594-36f2-42e1-9017-f4e9011de5a2"
-					(reference "R3")
-					(unit 1)
-				)
+					(reference "R2")
+					(unit 1)
+				)

Commit message: Added more clearance for mounting holes
Parts:
- H1, H2, H3, H4: footprint MountingHole:MountingHole_2.5mm -> MountingHole:MountingHole_4.5mm
Changed lines of the file:
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@@
 			)
 		)
-		(property "Footprint" "MountingHole:MountingHole_2.5mm"
+		(property "Footprint" "MountingHole:MountingHole_4.5mm"
 			(at 82.55 172.72 0)
 			(effects
@@
 			)
 		)
-		(property "Footprint" "MountingHole:MountingHole_2.5mm"
+		(property "Footprint" "MountingHole:MountingHole_4.5mm"
 			(at 105.41 172.72 0)
 			(effects
@@
 			)
 		)
-		(property "Footprint" "MountingHole:MountingHole_2.5mm"
+		(property "Footprint" "MountingHole:MountingHole_4.5mm"
 			(at 105.41 179.07 0)
 			(effects
@@
 			)
 		)
-		(property "Footprint" "MountingHole:MountingHole_2.5mm"
+		(property "Footprint" "MountingHole:MountingHole_4.5mm"
 			(at 82.55 179.07 0)
 			(effects
